File: hw/laser_driver.sch (EAGLE design)
At the start: 10 parts, among them IC1 895-FT232RL, IC2 998-MIC5209-3.0YM, X1 798-ZX62RD-AB-5P8

Commit message: Change connector to terminal block
Parts:
- JP1: value (none) -> 651-5442251; device SparkFun-Connectors:M03JST-PTH -> SparkFun-Connectors:M03SCREW
Changed lines of the file:
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@@
 <part name="GND7" library="SparkFun" deviceset="GND" device=""/>
 <part name="U$3" library="SparkFun" deviceset="5V" device=""/>
-<part name="JP1" library="SparkFun-Connectors" deviceset="M03" device="JST-PTH"/>
 <part name="+3V32" library="supply1" deviceset="+3V3" device="" value="+3V"/>
 <part name="GND4" library="supply1" deviceset="GND" device=""/>
@@
 <part name="GND10" library="SparkFun" deviceset="GND" device=""/>
 <part name="LOGO1" library="SparkFun-Aesthetics" deviceset="OSHW-LOGO" device="S" value="OSHW-LOGOS"/>
+<part name="JP1" library="SparkFun-Connectors" deviceset="M03" device="SCREW" value="651-5442251"/>
 </parts>
 <sheets>
@@
 <attribute name="VALUE" x="34.544" y="59.436" size="1.778" layer="96"/>
 </instance>
-<instance part="JP1" gate="G$1" x="220.98" y="43.18" rot="R180"/>
 <instance part="+3V32" gate="G$1" x="175.26" y="50.8" smashed="yes">
 <attribute name="VALUE" x="172.72" y="50.8" size="1.778" layer="96"/>
@@
 </instance>
 <instance part="LOGO1" gate="G$1" x="106.68" y="-10.16"/>
+<instance part="JP1" gate="G$1" x="220.98" y="43.18" smashed="yes" rot="R180">
+<attribute name="NAME" x="223.52" y="37.338" size="1.778" layer="95" rot="R180"/>
+</instance>
 </instances>
 <busses>
@@
 </segment>
 <segment>
-<pinref part="JP1" gate="G$1" pin="3"/>
 <wire x1="213.36" y1="40.64" x2="200.66" y2="40.64" width="0.1524" layer="91"/>
 <pinref part="GND10" gate="1" pin="GND"/>
 <wire x1="200.66" y1="38.1" x2="200.66" y2="40.64" width="0.1524" layer="91"/>
+<pinref part="JP1" gate="G$1" pin="3"/>
 </segment>
 </net>
@@
 </segment>
 <segment>
-<pinref part="JP1" gate="G$1" pin="2"/>
 <wire x1="213.36" y1="43.18" x2="200.66" y2="43.18" width="0.1524" layer="91"/>
 <label x="200.66" y="43.18" size="1.778" layer="95"/>
+<pinref part="JP1" gate="G$1" pin="2"/>
 </segment>
 </net>
@@
 </segment>
 <segment>
-<pinref part="JP1" gate="G$1" pin="1"/>
 <wire x1="213.36" y1="45.72" x2="200.66" y2="45.72" width="0.1524" layer="91"/>
 <pinref part="+3V1" gate="G$1" pin="+3V3"/>
 <wire x1="200.66" y1="48.26" x2="200.66" y2="45.72" width="0.1524" layer="91"/>
-</segment>
-</net>
+<pinref part="JP1" gate="G$1" pin="1"/>
+</segment>
+</net>

Commit message: Fix noise cap for the regulator
Parts:
- C6: value C1608X5R1C106M080AB -> VJ0603A471KXQPW1BC
Changed lines of the file:
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@@
 <part name="C4" library="SparkFun-Passives" deviceset="CAP" device="0603-CAP" value="C1608X5R1C106M080AB"/>
 <part name="IC2" library="v-reg-micrel" deviceset="MIC5219BMM" device="" value="998-MIC5209-3.0YM"/>
-<part name="C6" library="SparkFun-Passives" deviceset="CAP" device="0603-CAP" value="C1608X5R1C106M080AB"/>
+<part name="C6" library="SparkFun-Passives" deviceset="CAP" device="0603-CAP" value="VJ0603A471KXQPW1BC"/>
 <part name="GND6" library="supply1" deviceset="GND" device=""/>
 <part name="GND3" library="supply1" deviceset="GND" device=""/>

Commit message: Fix part numbers for regulator and usb plug. Fix disconnectoed ground pin (4) which was a really stupid mistake...
Parts:
- IC2: value 998-MIC5209-3.0YM -> 998-MIC5219-3.0YMM
Changed lines of the file:
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@@
 <part name="C3" library="SparkFun-Passives" deviceset="CAP" device="0603-CAP" value="C1608X5R1C106M080AB"/>
 <part name="C4" library="SparkFun-Passives" deviceset="CAP" device="0603-CAP" value="C1608X5R1C106M080AB"/>
-<part name="IC2" library="v-reg-micrel" deviceset="MIC5219BMM" device="" value="998-MIC5209-3.0YM"/>
+<part name="IC2" library="v-reg-micrel" deviceset="MIC5219BMM" device="" value="998-MIC5219-3.0YMM"/>
 <part name="C6" library="SparkFun-Passives" deviceset="CAP" device="0603-CAP" value="VJ0603A471KXQPW1BC"/>
 <part name="GND6" library="supply1" deviceset="GND" device=""/>
